File: Circuit/trinkle.sch (KiCad schematic (older format))
At the start: 12 parts, among them IC1 ATTINY84A-SS, P1 ISCP, P2 CONN_7, P3 CONN_7, SW1 SW_PUSH

Commit message: Added pdf of schematic
Parts:
- C2: value 10u -> 1u
Changed lines of the file:
@@
 LIBS:contrib
 LIBS:valves
-LIBS:hd44780_backpack
+LIBS:trinkle-cache
 EELAYER 27 0
 EELAYER END
@@
 Sheet 1 1
 Title ""
-Date "2 jul 2014"
-Rev ""
+Date "15 jul 2014"
+Rev "1.1"
 Comp ""
 Comment1 ""
@@
 $EndComp
 $Comp
-L +5V #PWR2
+L +5V #PWR01
 U 1 1 53B3E7AC
 P 2750 2900
-F 0 "#PWR2" H 2750 2990 20  0001 C CNN
+F 0 "#PWR01" H 2750 2990 20  0001 C CNN
 F 1 "+5V" H 2750 2990 30  0000 C CNN
 F 2 "" H 2750 2900 60  0000 C CNN
@@
 $EndComp
 $Comp
-L GND #PWR1
+L GND #PWR02
 U 1 1 53B3E7C0
 P 2700 3300
-F 0 "#PWR1" H 2700 3300 30  0001 C CNN
+F 0 "#PWR02" H 2700 3300 30  0001 C CNN
 F 1 "GND" H 2700 3230 30  0001 C CNN
 F 2 "" H 2700 3300 60  0000 C CNN
@@
 P 2950 3100
 F 0 "C2" H 2950 3200 40  0000 L CNN
-F 1 "10u" H 2956 3015 40  0000 L CNN
+F 1 "1u" H 2956 3015 40  0000 L CNN
 F 2 "~" H 2988 2950 30  0000 C CNN
 F 3 "~" H 2950 3100 60  0000 C CNN
@@
 $EndComp
 $Comp
-L GND #PWR7
+L GND #PWR03
 U 1 1 53B3E940
 P 6900 1900
-F 0 "#PWR7" H 6900 1900 30  0001 C CNN
+F 0 "#PWR03" H 6900 1900 30  0001 C CNN
 F 1 "GND" H 6900 1830 30  0001 C CNN
 F 2 "" H 6900 1900 60  0000 C CNN
@@
 	5650 2650 6950 2650
 $Comp
-L +5V #PWR8
+L +5V #PWR04
 U 1 1 53B3EA7F
 P 6950 3900
-F 0 "#PWR8" H 6950 3990 20  0001 C CNN
+F 0 "#PWR04" H 6950 3990 20  0001 C CNN
 F 1 "+5V" H 6950 3990 30  0000 C CNN
 F 2 "" H 6950 3900 60  0000 C CNN
@@
 	6500 3350 6950 3350
 $Comp
-L +5V #PWR6
+L +5V #PWR05
 U 1 1 53B3EC75
 P 6500 1050
-F 0 "#PWR6" H 6500 1140 20  0001 C CNN
+F 0 "#PWR05" H 6500 1140 20  0001 C CNN
 F 1 "+5V" H 6500 1140 30  0000 C CNN
 F 2 "" H 6500 1050 60  0000 C CNN
@@
 $EndComp
 $Comp
-L GND #PWR5
+L GND #PWR06
 U 1 1 53B3EF92
 P 5850 4800
-F 0 "#PWR5" H 5850 4800 30  0001 C CNN
+F 0 "#PWR06" H 5850 4800 30  0001 C CNN
 F 1 "GND" H 5850 4730 30  0001 C CNN
 F 2 "" H 5850 4800 60  0000 C CNN
@@
 $EndComp
 $Comp
-L +5V #PWR3
+L +5V #PWR07
 U 1 1 53B3F0F7
 P 5150 1600
-F 0 "#PWR3" H 5150 1690 20  0001 C CNN
+F 0 "#PWR07" H 5150 1690 20  0001 C CNN
 F 1 "+5V" H 5150 1690 30  0000 C CNN
 F 2 "" H 5150 1600 60  0000 C CNN
@@
 $EndComp
 $Comp
-L GND #PWR4
+L GND #PWR08
 U 1 1 53B3F1B7
 P 5150 1850
-F 0 "#PWR4" H 5150 1850 30  0001 C CNN
+F 0 "#PWR08" H 5150 1850 30  0001 C CNN
 F 1 "GND" H 5150 1780 30  0001 C CNN
 F 2 "" H 5150 1850 60  0000 C CNN

Commit message: Added usb port
Snap off capable usb port section
Parts:
- added CON1: USB-MINI-B, symbol USB-MINI-B
- added D3, D4: DIODE, ~, symbol DIODE
- added P4: CONN_4, symbol CONN_4
- added R4: 1k, ~, symbol R
- added R5, R6: 68, ~, symbol R
- D1: value LED -> PWR_LED
- D2: value LED -> D8_LED
Connections:
- net +5V: now also CON1.1 (VBUS), P4.4 (P4), R4.2
- net GND: now also CON1.5 (GND), D3.1 (A), D4.1 (A), P4.1 (P1)
- net at IC1.2 ((PCINT8/CLKI/XTAL1)PB0), P3.2 (P2): now also D4.2 (K), P4.3 (P3), R6.2
- net at IC1.3 ((PCINT9/XTAL2)PB1), P3.3 (P3): now also P4.2 (P2), R5.2
- new net: CON1.2 (D-), R4.1, R6.1
- new net: CON1.3 (D+), D3.2 (K), R5.1
Changed lines of the file:
@@
 LIBS:contrib
 LIBS:valves
+LIBS:hd44780_backpack
 LIBS:trinkle-cache
 EELAYER 27 0
@@
 Sheet 1 1
 Title ""
-Date "15 jul 2014"
+Date "31 aug 2014"
 Rev "1.1"
 Comp ""
@@
 P 3200 2900
 F 0 "D1" H 3200 3000 50  0000 C CNN
-F 1 "LED" H 3200 2800 50  0000 C CNN
+F 1 "PWR_LED" H 3200 2800 50  0000 C CNN
 F 2 "~" H 3200 2900 60  0000 C CNN
 F 3 "~" H 3200 2900 60  0000 C CNN
@@
 P 5850 4100
 F 0 "D2" H 5850 4200 50  0000 C CNN
-F 1 "LED" H 5850 4000 50  0000 C CNN
+F 1 "D8_LED" H 5850 4000 50  0000 C CNN
 F 2 "~" H 5850 4100 60  0000 C CNN
 F 3 "~" H 5850 4100 60  0000 C CNN
@@
 	5800 1850 5800 1600
 Connection ~ 5800 1600
+$Comp
+L USB-MINI-B CON1
+U 1 1 53F1DD1C
+P 4050 5100
+F 0 "CON1" H 3800 5550 60  0000 C CNN
+F 1 "USB-MINI-B" H 4000 4600 60  0000 C CNN
+F 2 "" H 4050 5100 60  0000 C CNN
+F 3 "" H 4050 5100 60  0000 C CNN
+	1    4050 5100
+	-1   0    0    1
+$EndComp
+$Comp
+L GND #PWR09
+U 1 1 54031E7D
+P 4600 4450
+F 0 "#PWR09" H 4600 4450 30  0001 C CNN
+F 1 "GND" H 4600 4380 30  0001 C CNN
+F 2 "" H 4600 4450 60  0000 C CNN
+F 3 "" H 4600 4450 60  0000 C CNN
+	1    4600 4450
+	-1   0    0    1
+$EndComp
+Wire Wire Line
+	4600 4800 4600 4450
+$Comp
+L +5V #PWR010
+U 1 1 540320C9
+P 4850 5900
+F 0 "#PWR010" H 4850 5990 20  0001 C CNN
+F 1 "+5V" H 4850 5990 30  0000 C CNN
+F 2 "" H 4850 5900 60  0000 C CNN
+F 3 "" H 4850 5900 60  0000 C CNN
+	1    4850 5900
+	-1   0    0    1
+$EndComp
+$Comp
+L R R4
+U 1 1 54032140
+P 4850 5650
+F 0 "R4" V 4930 5650 40  0000 C CNN
+F 1 "1k" V 4857 5651 40  0000 C CNN
+F 2 "~" V 4780 5650 30  0000 C CNN
+F 3 "~" H 4850 5650 30  0000 C CNN
+	1    4850 5650
+	1    0    0    -1
+$EndComp
+Wire Wire Line
+	4850 5900 4600 5900
+Wire Wire Line
+	4600 5900 4600 5400
+Connection ~ 4850 5900
+Connection ~ 4850 5250
+Wire Wire Line
+	4850 5400 4850 5250
+Wire Wire Line
+	5650 5250 5650 3450
+Connection ~ 5650 3450
+Wire Wire Line
+	5550 5100 5550 3550
+Connection ~ 5550 3550
+$Comp
+L R R6
+U 1 1 540322DD
+P 5400 5250
+F 0 "R6" V 5480 5250 40  0000 C CNN
+F 1 "68" V 5407 5251 40  0000 C CNN
+F 2 "~" V 5330 5250 30  0000 C CNN
+F 3 "~" H 5400 5250 30  0000 C CNN
+	1    5400 5250
+	0    -1   -1   0
+$EndComp
+$Comp
+L R R5
+U 1 1 54032305
+P 4950 5100
+F 0 "R5" V 5030 5100 40  0000 C CNN
+F 1 "68" V 4957 5101 40  0000 C CNN
+F 2 "~" V 4880 5100 30  0000 C CNN
+F 3 "~" H 4950 5100 30  0000 C CNN
+	1    4950 5100
+	0    -1   -1   0
+$EndComp
+Wire Wire Line
+	4600 5250 5150 5250
+Wire Wire Line
+	4700 5100 4600 5100
+$Comp
+L DIODE D3
+U 1 1 540324BD
+P 4850 4700
+F 0 "D3" H 4850 4800 40  0000 C CNN
+F 1 "DIODE" H 4850 4600 40  0000 C CNN
+F 2 "~" H 4850 4700 60  0000 C CNN
+F 3 "~" H 4850 4700 60  0000 C CNN
+	1    4850 4700
+	0    1    1    0
+$EndComp
+$Comp
+L DIODE D4
+U 1 1 540324EE
+P 5150 4700
+F 0 "D4" H 5150 4800 40  0000 C CNN
+F 1 "DIODE" H 5150 4600 40  0000 C CNN
+F 2 "~" H 5150 4700 60  0000 C CNN
+F 3 "~" H 5150 4700 60  0000 C CNN
+	1    5150 4700
+	0    1    1    0
+$EndComp
+Wire Wire Line
+	4600 4500 5150 4500
+Connection ~ 4600 4500
+Connection ~ 4850 4500
+Wire Wire Line
+	4850 4900 4700 4900
+Wire Wire Line
+	4700 4900 4700 5100
+Connection ~ 5650 4900
+Connection ~ 4700 5100
+Connection ~ 5150 4500
+Connection ~ 5200 5100
+Connection ~ 5150 4900
+Connection ~ 4850 4900
+$Comp
+L CONN_4 P4
+U 1 1 5403274C
+P 6700 5050
+F 0 "P4" V 6650 5050 50  0000 C CNN
+F 1 "CONN_4" V 6750 5050 50  0000 C CNN
+F 2 "" H 6700 5050 60  0000 C CNN
+F 3 "" H 6700 5050 60  0000 C CNN
+	1    6700 5050
+	1    0    0    -1
+$EndComp
+$Comp
+L GND #PWR011
+U 1 1 54032797
+P 6350 4700
+F 0 "#PWR011" H 6350 4700 30  0001 C CNN
+F 1 "GND" H 6350 4630 30  0001 C CNN
+F 2 "" H 6350 4700 60  0000 C CNN
+F 3 "" H 6350 4700 60  0000 C CNN
+	1    6350 4700
+	-1   0    0    1
+$EndComp
+Wire Wire Line
+	6350 4900 6350 4700
+$Comp
+L +5V #PWR012
+U 1 1 54032812
+P 6350 5300
+F 0 "#PWR012" H 6350 5390 20  0001 C CNN
+F 1 "+5V" H 6350 5390 30  0000 C CNN
+F 2 "" H 6350 5300 60  0000 C CNN
+F 3 "" H 6350 5300 60  0000 C CNN
+	1    6350 5300
+	-1   0    0    1
+$EndComp
+Wire Wire Line
+	6350 5300 6350 5200
+Connection ~ 5550 5100
+Wire Wire Line
+	5200 5100 5750 5100
+Wire Wire Line
+	5150 4900 5800 4900
+Wire Wire Line
+	5800 4900 5800 5100
+Wire Wire Line
+	5800 5100 6350 5100
+Wire Wire Line
+	5750 5100 5750 5000
+Wire Wire Line
+	5750 5000 6350 5000
 $EndSCHEMATC
